File: hardware/devboard/dc26-dev-board/dc26-dev-board.sch (EAGLE design)
At the start: 51 parts, among them IC1 STM32F411RET6, IC10 APA104, IC11 APA104, IC12 APA104, IC13 APA104, IC14 APA104, IC15 APA104, IC16 APA104, IC2 APA104, IC3 APA104, IC4 APA104, IC5 APA104, IC6 APA104, IC7 APA104, IC8 APA104, IC9 APA104, U1 ESP-WROOM-32, Y1 ABL-8.000MHZ-B2

Commit message: all errors gone from schema
Parts:
- removed 3.3V-REGULATOR: BU33SD5WG-TR, dc-26:BU33SD5WG-TR
- removed IC10, IC11, IC12, IC13, IC14, IC15, IC16, IC2, IC3, IC4, IC5, IC6, IC7, IC8, IC9: APA104, APA104:APA104
- added APA1, APA10, APA11, APA12, APA13, APA14, APA15, APA16, APA17, APA18, APA19, APA2, APA20, APA3, APA4, APA5, APA6, APA7, APA8, APA9: APA104, APA104:APA104
- added C14, C29, C30, C31, C32, C33, C34, C35, C36, C37, C38, C39, C40, C41, C42, C43, C44, C45, C46, C47: 15pf, dc-26:C-USC0805
- added C15, C16: 20pf, dc-26:C-USC0805
- added C17: 4.7uF, dc-26:C-USC0805
- added M10: STM32-Breakout-2, dc-26:M10SILK_FEMALE_PTH
- added PS1: LD39050PU33R, dc-26:LD39050PU33R
- CN1: value (none) -> JST
Connections:
- removed net ESP-TXD0: ESP32-PROGRAM-HEADER.TX
- removed net N$4: 3.3V-REGULATOR.VIN, C3.2, RESETTABLE-FUSE.2, U$5.1
- removed net N$6: 3.3V-REGULATOR.STBY, U$5.C
- removed net VBAT: IC1.VBAT
- removed net VDD1: IC1.VDD(1)
- removed net VDD3: IC1.VDD(3)
- removed net VDD4: IC1.VDD(4)
- removed net VSS2: IC1.VSS(2)
- new net BOOT0: IC1.BOOT0, STM32-BREAKOUT.9
- new net CLK: ESP-BREAKOUT.20, U1.CLK
- new net CMD: ESP-BREAKOUT.19, U1.CMD
- new net IO14: ESP-BREAKOUT.13, U1.IO14
- new net IO16: ESP-BREAKOUT.27, U1.IO16
- new net IO17: ESP-BREAKOUT.28, U1.IO17
- new net IO18: ESP-BREAKOUT.30, U1.IO18
- new net IO19: ESP-BREAKOUT.31, U1.IO19
- new net IO22: ESP-BREAKOUT.36, U1.IO22
- new net IO23: ESP-BREAKOUT.37, U1.IO23
- new net IO25: ESP-BREAKOUT.10, U1.IO25
- new net IO26: ESP-BREAKOUT.11, U1.IO26
- new net IO27: ESP-BREAKOUT.12, U1.IO27
- new net IO32: ESP-BREAKOUT.8, U1.IO32
- new net IO33: ESP-BREAKOUT.9, U1.IO33
- new net IO34: ESP-BREAKOUT.6, U1.IO34
- new net IO35: ESP-BREAKOUT.7, U1.IO35
- new net IO4: ESP-BREAKOUT.26, U1.IO4
- new net IO5: ESP-BREAKOUT.29, U1.IO5
- new net N$20: C17.1, IC1.VCAP_1
- new net N$21: APA17.DIN, APA18.DOUT
- new net N$22: APA4.DOUT, APA5.DIN
- new net N$23: APA8.DOUT, APA9.DIN
- new net N$24: APA12.DOUT, APA16.DIN
- new net N$25: APA13.DOUT, APA20.DIN
- new net NRST: IC1.NRST, STM32-BREAKOUT.11
- new net PA0: IC1.PA0, STM32-BREAKOUT.23
- new net PA1: IC1.PA1, STM32-BREAKOUT.25
- new net PA10: IC1.PA10, STM32-BREAKOUT.12
- new net PA15: IC1.PA15, STM32-BREAKOUT.10
- new net PA2: IC1.PA2, STM32-BREAKOUT.27
- new net PA3: IC1.PA3, STM32-BREAKOUT.29
- new net PA4: IC1.PA4, STM32-BREAKOUT.31
- new net PA5: IC1.PA5, STM32-BREAKOUT.33
- new net PA6: IC1.PA6, STM32-BREAKOUT.35
- new net PA7: IC1.PA7, STM32-BREAKOUT.37
- new net PA9: IC1.PA9, STM32-BREAKOUT.14
- new net PB0: IC1.PB0, STM32-BREAKOUT.38
- new net PB1: IC1.PB1, STM32-BREAKOUT.36
- new net PB13: IC1.PB13, STM32-BREAKOUT.21
- new net PB14: IC1.PB14, STM32-BREAKOUT.28
- new net PB15: IC1.PB15, STM32-BREAKOUT.26
- new net PB3: IC1.PB3, M10.2
- new net PB4: IC1.PB4, M10.3
- new net PB5: IC1.PB5, M10.4
- new net PB6: IC1.PB6, M10.5
- new net PB7: IC1.PB7, M10.6
- new net PB8: IC1.PB8, M10.7
- new net PB9: IC1.PB9, M10.8
- new net PC10: IC1.PC10, STM32-BREAKOUT.8
- new net PC13: IC1.PC13, STM32-BREAKOUT.3
- new net PC14: IC1.PC14-OSC32_IN, STM32-BREAKOUT.5
- new net PC15: IC1.PC15-OSC32_OUT, STM32-BREAKOUT.7
- new net PC2: IC1.PC2, STM32-BREAKOUT.17
- new net PC6: IC1.PC6, STM32-BREAKOUT.24
- new net PC7: IC1.PC7, STM32-BREAKOUT.22
- new net PC8: IC1.PC8, STM32-BREAKOUT.20
- new net PC9: IC1.PC9, STM32-BREAKOUT.18
- new net SD1: ESP-BREAKOUT.22, U1.SD1
- new net SD2: ESP-BREAKOUT.17, U1.SD2
- new net SD3: ESP-BREAKOUT.18, U1.SD3
- new net SDO: ESP-BREAKOUT.21, U1.SDO
- new net SENSOR_VN: ESP-BREAKOUT.5, U1.SENSOR_VN
- new net SENSOR_VP: ESP-BREAKOUT.4, U1.SENSOR_VP
- new net VIN: C3.2, PS1.VIN, RESETTABLE-FUSE.2, U$5.1
- new net VIN-EN: PS1.EN, U$5.C
- net ESP-IO0: now also ESP-BREAKOUT.25
- net ESP-RX0: now also ESP-BREAKOUT.34
- net ESP-TX0: now also ESP-BREAKOUT.35, ESP32-PROGRAM-HEADER.TX
- net ESP_CS: now also ESP-BREAKOUT.33, M10.1, U1.IO21
- net GND: now also APA1.VSS, APA10.VSS, APA11.VSS, APA12.VSS, APA13.VSS, APA14.VSS, APA15.VSS, APA16.VSS, APA17.VSS, APA18.VSS, APA19.VSS, APA2.VSS, APA20.VSS, APA3.VSS, APA4.VSS, APA5.VSS, APA6.VSS, APA7.VSS, APA8.VSS, APA9.VSS, C14.2, C15.1, C16.1, C17.2, C29.2, C30.2, C31.2, C32.2, C33.2, C34.2, C35.2, C36.2, C37.2, C38.2, C39.2, C40.2, C41.2, C42.2, C43.2, C44.2, C45.2, C46.2, C47.2, ESP-BREAKOUT.1, ESP-BREAKOUT.15, ESP-BREAKOUT.24, ESP-BREAKOUT.38, IC1.VSS(2), M10.9, PS1.GND, PS1.PAD, STM32-BREAKOUT.2; no longer 3.3V-REGULATOR.GND, IC1.VDD(2), IC10.VSS, IC11.VSS, IC12.VSS, IC13.VSS, IC14.VSS, IC15.VSS, IC16.VSS, IC2.VSS, IC3.VSS, IC4.VSS, IC5.VSS, IC6.VSS, IC7.VSS, IC8.VSS, IC9.VSS
- net GPIO_APA104_DATA: now also APA1.DIN, STM32-BREAKOUT.16; no longer IC15.DIN
- net LCD_BACKLIGHT: now also STM32-BREAKOUT.34
- net LCD_CS: now also STM32-BREAKOUT.15
- net LCD_DATA_CMD: now also STM32-BREAKOUT.13
- net LCD_RESET: now also STM32-BREAKOUT.40
- net N$10: now also APA6.DOUT, APA7.DIN; no longer IC10.DOUT, IC14.DIN
- net N$11: now also APA7.DOUT, APA8.DIN; no longer IC14.DOUT, IC7.DIN
- net N$12: now also APA10.DIN, APA9.DOUT; no longer IC13.DIN, IC7.DOUT
- net N$13: now also APA10.DOUT, APA11.DIN; no longer IC13.DOUT, IC6.DIN
- net N$14: now also APA11.DOUT, APA12.DIN; no longer IC12.DIN, IC6.DOUT
- net N$15: now also APA15.DIN, APA16.DOUT; no longer IC12.DOUT, IC5.DIN
- net N$16: now also APA14.DIN, APA15.DOUT; no longer IC4.DIN, IC5.DOUT
- net N$17: now also APA13.DIN, APA14.DOUT; no longer IC11.DIN, IC4.DOUT
- net N$18: now also APA19.DIN, APA20.DOUT; no longer IC11.DOUT, IC3.DIN
- net N$19: now also APA18.DIN, APA19.DOUT; no longer IC2.DIN, IC3.DOUT
- net N$5: now also APA1.DOUT, APA2.DIN; no longer IC15.DOUT, IC8.DIN
- net N$7: now also APA2.DOUT, APA3.DIN; no longer IC8.DOUT, IC9.DIN
- net N$8: now also APA3.DOUT, APA4.DIN; no longer IC16.DIN, IC9.DOUT
- net N$9: now also APA5.DOUT, APA6.DIN; no longer IC10.DIN, IC16.DOUT
- net OSC_IN: now also C16.2
- net OSC_OUT: now also C15.2
- net SD_CS: now also STM32-BREAKOUT.39
- net SPI2_LCD_MOSI: now also STM32-BREAKOUT.19
- net SPI2_LCD_SCK: now also STM32-BREAKOUT.32
- net SPI3_ESP_MISO: now also ESP-BREAKOUT.16, STM32-BREAKOUT.6, U1.IO13
- net SPI3_ESP_MOSI: now also ESP-BREAKOUT.14, STM32-BREAKOUT.4, U1.IO12
- net SPI3_ESP_SCK: now also ESP-BREAKOUT.23, STM32-BREAKOUT.30, U1.IO15
- net VCC: now also C13.1, ESP-BREAKOUT.2, IC1.VBAT, IC1.VDD(1), IC1.VDD(2), IC1.VDD(3), IC1.VDD(4), M10.10, PS1.VOUT, STM32-BREAKOUT.1; no longer 3.3V-REGULATOR.VOUT, C11.1, C12.1, FB1.2
- net VCC1: now also APA1.VDD, APA10.VDD, APA11.VDD, APA12.VDD, APA13.VDD, APA14.VDD, APA15.VDD, APA16.VDD, APA17.VDD, APA18.VDD, APA19.VDD, APA2.VDD, APA20.VDD, APA3.VDD, APA4.VDD, APA5.VDD, APA6.VDD, APA7.VDD, APA8.VDD, APA9.VDD, C14.1, C29.1, C30.1, C31.1, C32.1, C33.1, C34.1, C35.1, C36.1, C37.1, C38.1, C39.1, C40.1, C41.1, C42.1, C43.1, C44.1, C45.1, C46.1, C47.1; no longer IC10.VDD, IC11.VDD, IC12.VDD, IC13.VDD, IC14.VDD, IC15.VDD, IC16.VDD, IC2.VDD, IC3.VDD, IC4.VDD, IC5.VDD, IC6.VDD, IC7.VDD, IC8.VDD, IC9.VDD
- net VDDA: now also C11.1, C12.1, FB1.2
Other:
- note added: "3.7V From Battery Out"
- note added: "5V ST-Link In"
- note added: "APA104's need at least 3.5V hence why we connect to VCC1"
- note added: "ESP-WROOM-32"
- note added: "This is correct: SD Card reader and ESP 32 share the same SPI"
- note added: "VBAT"
- note added: "VCC0 = 5V VCC 1 = 3.7 V VCC = 3.3V"
- note added: "VDD1"
- note added: "VDD2"
- note added: "VDD3"
- note added: "VDD4"
- note removed: "APA104's need at least 3.5V"

Commit message: added a user button and a button to reset
Parts:
- added C18, C19: 100nF, dc-26:C-USC0805
- added R5: 10K, dc-26:RESISTOR0805-RES
- added R6: 100, dc-26:RESISTOR0805-RES
- added R7, R8: 4K7, dc-26:RESISTOR0805-RES
- added U$6: MJTP1243, dc-26:SWITCH_TACTILETACTILE-2PIN-NARROW
- added USERBUTTON: UserButton, dc-26:SWITCH_TACTILETACTILE-2PIN-NARROW
Connections:
- new net N$4: C19.2, R6.2
- net BOOT0: now also R5.1
- net GND: now also C18.2, R5.2, R6.1, U$6.A, USERBUTTON.A
- net NRST: now also C18.1, R8.2, U$6.C
- net PC13: now also C19.1, R7.2, USERBUTTON.C
- net VCC: now also R7.1, R8.1
Other:
- note added: "Power"
