File: hardware/devboard/dc26-dev-board/dc26-dev-board.sch (EAGLE design)
At the start: 88 parts, among them CN1 JST, IC1 STM32F411RET6, M10 STM32-Breakout-2, U1 ESP-WROOM-32, Y1 ABL-8.000MHZ-B2

Commit message: Autoroute (#1)
* inital board layout

* first auto route

* auto routed boardwith some minor vcc changes by hand.

* minor fixed of part naming and added todo file

* added R9 to crystal
moved logo and DN to tslik and bsilk layers
Parts:
- added LINK1: STLINK-V2-CONNECTOR, dc-26:STLINK-V2-CONNECTOR
- added R9: 1M, dc-26:RESISTOR0805-RES
- added U$3: DARKNET_DD, dc-26:DARKNET_DD
- added USB: DX4R005JJ2DX4R005JJ2, dc-26:DX4R005JJ2DX4R005JJ2
- P1: value SWITCH_SPDT -> SSSS811101
- U$2: value DX4R005JJ2DX4R005JJ2 -> CMD_C0DE_LOGO; device dc-26:DX4R005JJ2DX4R005JJ2 -> dc-26:CMD_C0DE_LOGO
- U$4: value STLINK-V2-CONNECTOR -> DARKNET_NN; device dc-26:STLINK-V2-CONNECTOR -> dc-26:DARKNET_NN
- renumbered ESP32-PROGRAM-HEADER to ESP32PH, U$5 to P1, VOLTAGE_REG_1A_3.3V to VDO
Connections:
- net GND: now also LINK1.GND, P1.1, USB.GND; no longer U$2.GND, U$4.GND
- net OSC_IN: now also R9.2
- net OSC_OUT: now also R9.1
- net SYS_JTCK_SWCLK: now also LINK1.SWDCLK; no longer U$4.SWDCLK
- net SYS_JTMS_SWDIO: now also LINK1.SWDIO; no longer U$4.SWDIO
- net USB_DM: now also USB.D+; no longer U$2.D+
- net USB_DP: now also USB.D-; no longer U$2.D-
- net VCC0: now also LINK1.VCC, USB.+5V; no longer U$2.+5V, U$4.VCC
- net VIN: now also P1.2; no longer P1.1
