File: hardware/devboard/dc26-dev-board/dc26-dev-boardv3.sch (EAGLE design)
At the start: 100 parts, among them CN1 JST, IC1 STM32F411RET6, IC2 S2305TR, IC3 LDL112D33R, IC4 S2305TR, M10 STM32-Breakout-2, P1 SSSS811101, U1 ESP-WROOM-32, Y1 ABL-8.000MHZ-B2

Commit message: added new tvs diode after talking with bunni even made the part myself
Parts:
- removed IC2, IC4: S2305TR, dc-26:S2305TR
- added U$17: XBP15SRV05W-G, dc-26:XBP15SRV05W-G
- C2: value 4.7uf -> 4.7uF
- C3, C4: value 1uf -> 1uF
- LED2: value 3mm -> LED2-3MM
- renumbered IC1 to SOC1, U$1 to LCD1, U$10 to APA106-2, U$11 to APA106-3, U$12 to APA106-4, U$13 to APA106-5, U$14 to APA106-6, U$15 to OLED1, U$5 to APA102-2, U$6 to APA102-3, U$7 to APA102-4, U$8 to APA102-1, U$9 to APA106-1, U1 to SOC2
Connections:
- removed net I2C1_SCL: M10.5, OLED1.SCL, SOC1.PB6
- removed net I2C1_SDA: M10.6, OLED1.SDA, SOC1.PB7
- removed net IO18: ESP-BREAKOUT.30, SOC2.IO18
- removed net IO19: ESP-BREAKOUT.31, SOC2.IO19
- new net ESP_I2C_SCL: ESP-BREAKOUT.31, M10.5, OLED1.SCL, SOC1.PB6, SOC2.IO19
- new net ESP_I2C_SDA: ESP-BREAKOUT.30, M10.6, OLED1.SDA, SOC1.PB7, SOC2.IO18
- net GND: now also U$17.P2; no longer IC2.CATH1, IC2.CATH2, IC4.CATH1, IC4.CATH2
- net USB_DM: now also U$17.P6; no longer IC4.ANODE
- net USB_DP: now also U$17.P1; no longer IC2.ANODE
