File: hardware/devboard/dc26-dev-board/dc26.brd (EAGLE design)
At the start: 126 x 70 mm, 112 parts, among them CN1 JST, IC3 LDL112D33R, J1 DC26 Shitty AddOn, J2 DC26 Shitty AddOn, P1 SPDT_SSAJ120100, Y1 ABL-8.000MHZ-B2

Commit message: basics of sd card working still have work todo to get flatbuffers working Buttons now working
Parts:
- removed U$12: MACROFAB_LOGO, darknet_parts_library:MACROFAB_LOGO
Changed lines of the file:
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@@
 <?xml version="1.0" encoding="utf-8"?>
 <!DOCTYPE eagle SYSTEM "eagle.dtd">
-<eagle version="7.7.0">
+<eagle version="9.0.1">
 <drawing>
 <settings>
 <setting alwaysvectorfont="no"/>
+<setting keepoldvectorfont="yes"/>
 <setting verticaltext="up"/>
 </settings>
@@
 <param name="dpMaxLengthDifference" value="10mm"/>
 <param name="dpGapFactor" value="2.5"/>
-<param name="checkGrid" value="0"/>
 <param name="checkAngle" value="0"/>
 <param name="checkFont" value="1"/>
 <param name="checkRestrict" value="1"/>
+<param name="checkStop" value="0"/>
+<param name="checkValues" value="0"/>
 <param name="useDiameter" value="13"/>
 <param name="maxErrors" value="50"/>
@@
 <element name="U$10" library="darknet_parts_library" package="FIDUCIAL_CORNER" value="FIDUCIAL_DNCORNER" x="17.790296875" y="11.18275" smashed="yes" rot="R90"/>
 <element name="U$11" library="darknet_parts_library" package="FIDUCIAL_CORNER" value="FIDUCIAL_DNCORNER" x="18.52918125" y="60.22345" smashed="yes" rot="MR270"/>
-<element name="U$12" library="darknet_parts_library" package="MACROFAB_LOGO" value="MACROFAB_LOGO" x="66.242153125" y="57.38271875" smashed="yes"/>
 </elements>
 <signals>
